File: Attiny-console.kicad_sch (KiCad schematic)
At the start: 15 parts, among them J1 SSD1306, J2 UDPI programming port, J3 Extra pins, SW1 SW_LEFT, SW2 SW_RIGHT, SW3 power_SW, SW4 power_SW, U1 ATtiny1616-S, U2 ATtiny1616-M

Commit message: The layout looks good now
Parts:
- BT1: footprint (none) -> Battery:BatteryHolder_Keystone_1060_1x2032
- BZ1: footprint (none) -> Buzzer_Beeper:MagneticBuzzer_Kobitone_254-EMB84Q-RO
- D1: footprint (none) -> LED_SMD:LED_0603_1608Metric_Pad1.05x0.95mm_HandSolder
- J1: footprint (none) -> Connector_PinSocket_2.54mm:PinSocket_1x04_P2.54mm_Vertical
- J2: footprint (none) -> Connector_PinSocket_2.54mm:PinSocket_1x03_P2.54mm_Horizontal
- J3: footprint (none) -> Connector_PinSocket_2.54mm:PinSocket_2x03_P2.54mm_Vertical
- R1, R3: footprint (none) -> Resistor_THT:R_Axial_DIN0207_L6.3mm_D2.5mm_P10.16mm_Horizontal
- R2: footprint (none) -> Resistor_SMD:R_0805_2012Metric_Pad1.20x1.40mm_HandSolder
- SW1, SW2: footprint (none) -> Button_Switch_THT:SW_PUSH_6mm
- SW3, SW4: footprint (none) -> Button_Switch_THT:SW_Slide_SPDT_Angled_CK_OS102011MA1Q
Connections:
- net left: now also U1.2 (PA4), U2.5 (PA4); no longer U1.19 (PA3), U2.2 (PA3)
- net right: now also U1.19 (PA3), U2.2 (PA3); no longer U1.2 (PA4), U2.5 (PA4)
Changed lines of the file:
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@@
 	)
 	(label "right"
-		(at 71.12 41.91 180)
+		(at 71.12 39.37 180)
 		(effects
 			(font
@@
 	)
 	(label "left"
-		(at 69.85 132.08 180)
+		(at 69.85 134.62 180)
 		(effects
 			(font
@@
 	)
 	(label "right"
-		(at 69.85 134.62 180)
+		(at 69.85 132.08 180)
 		(effects
 			(font
@@
 	)
 	(label "left"
-		(at 71.12 39.37 180)
+		(at 71.12 41.91 180)
 		(effects
 			(font
@@
 			)
 		)
-		(property "Footprint" ""
+		(property "Footprint" "LED_SMD:LED_0603_1608Metric_Pad1.05x0.95mm_HandSolder"
 			(at 194.31 36.83 0)
 			(hide yes)
@@
 			)
 		)
-		(property "Footprint" ""
+		(property "Footprint" "Connector_PinSocket_2.54mm:PinSocket_2x03_P2.54mm_Vertical"
 			(at 128.27 158.75 0)
 			(hide yes)
@@
 			)
 		)
-		(property "Footprint" ""
+		(property "Footprint" "Resistor_SMD:R_0805_2012Metric_Pad1.20x1.40mm_HandSolder"
 			(at 205.74 38.608 90)
 			(hide yes)
@@
 			)
 		)
-		(property "Footprint" ""
+		(property "Footprint" "Buzzer_Beeper:MagneticBuzzer_Kobitone_254-EMB84Q-RO"
 			(at 244.475 109.22 90)
 			(hide yes)
@@
 			)
 		)
-		(property "Footprint" ""
+		(property "Footprint" "Button_Switch_THT:SW_PUSH_6mm"
 			(at 130.81 81.28 0)
 			(hide yes)
@@
 			)
 		)
-		(property "Footprint" ""
+		(property "Footprint" "Button_Switch_THT:SW_Slide_SPDT_Angled_CK_OS102011MA1Q"
 			(at 232.41 109.22 0)
 			(hide yes)
@@
 			)
 		)
-		(property "Footprint" ""
+		(property "Footprint" "Button_Switch_THT:SW_Slide_SPDT_Angled_CK_OS102011MA1Q"
 			(at 236.22 54.61 0)
 			(hide yes)
@@
 			)
 		)
-		(property "Footprint" ""
+		(property "Footprint" "Resistor_THT:R_Axial_DIN0207_L6.3mm_D2.5mm_P10.16mm_Horizontal"
 			(at 164.592 72.39 90)
 			(hide yes)
@@
 			)
 		)
-		(property "Footprint" ""
+		(property "Footprint" "Resistor_THT:R_Axial_DIN0207_L6.3mm_D2.5mm_P10.16mm_Horizontal"
 			(at 120.142 71.12 90)
 			(hide yes)
@@
 			)
 		)
-		(property "Footprint" ""
+		(property "Footprint" "Connector_PinSocket_2.54mm:PinSocket_1x03_P2.54mm_Horizontal"
 			(at 156.21 116.84 0)
 			(hide yes)
@@
 			)
 		)
-		(property "Footprint" ""
+		(property "Footprint" "Battery:BatteryHolder_Keystone_1060_1x2032"
 			(at 247.65 58.166 90)
 			(hide yes)
@@
 			)
 		)
-		(property "Footprint" ""
+		(property "Footprint" "Connector_PinSocket_2.54mm:PinSocket_1x04_P2.54mm_Vertical"
 			(at 151.13 46.99 0)
 			(hide yes)
@@
 			)
 		)
-		(property "Footprint" ""
+		(property "Footprint" "Button_Switch_THT:SW_PUSH_6mm"
 			(at 173.99 82.55 0)
 			(hide yes)

Commit message: Finishing the layout
Parts:
- R1, R3: footprint Resistor_THT:R_Axial_DIN0207_L6.3mm_D2.5mm_P10.16mm_Horizontal -> Resistor_THT:R_Axial_DIN0207_L6.3mm_D2.5mm_P7.62mm_Horizontal
Connections:
- net MOSI: now also J3.3 (Pin_3); no longer J3.6 (Pin_6)
- net buzz: now also U1.9 (PB2), U2.12 (PB2); no longer U1.8 (PB3), U2.11 (PB3)
- net left: now also U1.19 (PA3), U2.2 (PA3); no longer U1.2 (PA4), U2.5 (PA4)
- net right: now also U1.2 (PA4), U2.5 (PA4); no longer U1.19 (PA3), U2.2 (PA3)
- net pc0: now reaches U2.15 (PC0)
- net pc0: now also J3.5 (Pin_5), U1.12 (PC0)
- net pc1: now reaches U2.16 (PC1)
- net pc1: now also J3.6 (Pin_6), U1.13 (PC1)
- removed net pb4: J3.3 (Pin_3), U1.7 (PB4), U2.10 (PB4)
- removed net pb5: J3.5 (Pin_5), U1.6 (PB5), U2.9 (PB5)
Changed lines of the file:
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@@
 	)
 	(no_connect
-		(at 34.29 149.86)
+		(at 64.77 157.48)
+	)
+	(no_connect
+		(at 66.04 62.23)
 	)
 	(no_connect
@@
 	)
 	(no_connect
+		(at 66.04 64.77)
+	)
+	(no_connect
 		(at 66.04 49.53)
 	)
@@
 	)
 	(no_connect
-		(at 35.56 57.15)
+		(at 64.77 137.16)
 	)
 	(no_connect
-		(at 64.77 137.16)
-	)
-	(no_connect
-		(at 66.04 59.69)
+		(at 66.04 67.31)
 	)
 	(no_connect
@@
 	)
 	(no_connect
-		(at 34.29 147.32)
+		(at 35.56 59.69)
 	)
 	(no_connect
-		(at 35.56 59.69)
+		(at 64.77 160.02)
 	)
 	(no_connect
@@
 	)
 	(no_connect
-		(at 64.77 152.4)
-	)
-	(no_connect
-		(at 35.56 54.61)
+		(at 64.77 154.94)
 	)
 	(no_connect
@@
 	(wire
 		(pts
-			(xy 64.77 157.48) (xy 69.85 157.48)
-		)
-		(stroke
-			(width 0)
-			(type default)
-		)
-	)
-	(wire
-		(pts
 			(xy 64.77 127) (xy 69.85 127)
 		)
@@
 	(wire
 		(pts
-			(xy 64.77 160.02) (xy 69.85 160.02)
-		)
-		(stroke
-			(width 0)
-			(type default)
-		)
-	)
-	(wire
-		(pts
 			(xy 146.05 116.84) (xy 151.13 116.84)
 		)
@@
 	(wire
 		(pts
-			(xy 66.04 67.31) (xy 71.12 67.31)
+			(xy 30.48 57.15) (xy 35.56 57.15)
 		)
 		(stroke
@@
 	(wire
 		(pts
-			(xy 66.04 64.77) (xy 71.12 64.77)
+			(xy 30.48 54.61) (xy 35.56 54.61)
 		)
 		(stroke
@@
 	(wire
 		(pts
-			(xy 66.04 62.23) (xy 71.12 62.23)
+			(xy 66.04 59.69) (xy 71.12 59.69)
 		)
 		(stroke
@@
 	(wire
 		(pts
+			(xy 29.21 149.86) (xy 34.29 149.86)
+		)
+		(stroke
+			(width 0)
+			(type default)
+		)
+	)
+	(wire
+		(pts
 			(xy 64.77 129.54) (xy 69.85 129.54)
 		)
@@
 	(wire
 		(pts
-			(xy 64.77 154.94) (xy 69.85 154.94)
+			(xy 64.77 152.4) (xy 69.85 152.4)
 		)
 		(stroke
@@
 		(pts
 			(xy 64.77 124.46) (xy 69.85 124.46)
+		)
+		(stroke
+			(width 0)
+			(type default)
+		)
+	)
+	(wire
+		(pts
+			(xy 29.21 147.32) (xy 34.29 147.32)
 		)
 		(stroke
@@
 		)
 	)
+	(label "pc1"
+		(at 29.21 149.86 0)
+		(effects
+			(font
+				(size 1.27 1.27)
+			)
+			(justify left bottom)
+		)
+	)
 	(label "SCL"
 		(at 71.12 54.61 180)
@@
 	)
 	(label "right"
-		(at 71.12 39.37 180)
+		(at 71.12 41.91 180)
 		(effects
 			(font
@@
 	)
 	(label "buzz"
-		(at 71.12 62.23 180)
+		(at 71.12 59.69 180)
 		(effects
 			(font
@@
 		)
 	)
+	(label "pc0"
+		(at 29.21 147.32 0)
+		(effects
+			(font
+				(size 1.27 1.27)
+			)
+			(justify left bottom)
+		)
+	)
 	(label "buzz"
-		(at 69.85 154.94 180)
+		(at 69.85 152.4 180)
 		(effects
 			(font
@@
 		)
 	)
-	(label "pb5"
-		(at 71.12 67.31 180)
-		(effects
-			(font
-				(size 1.27 1.27)
-			)
-			(justify right bottom)
+	(label "pc1"
+		(at 30.48 57.15 0)
+		(effects
+			(font
+				(size 1.27 1.27)
+			)
+			(justify left bottom)
 		)
 	)
@@
 		)
 	)
-	(label "pb5"
-		(at 116.84 161.29 0)
+	(label "pc1"
+		(at 142.24 161.29 180)
+		(effects
+			(font
+				(size 1.27 1.27)
+			)
+			(justify right bottom)
+		)
+	)
+	(label "pc0"
+		(at 30.48 54.61 0)
 		(effects
 			(font
@@
 			)
 			(justify left bottom)
-		)
-	)
-	(label "pb4"
-		(at 71.12 64.77 180)
-		(effects
-			(font
-				(size 1.27 1.27)
-			)
-			(justify right bottom)
 		)
 	)
@@
 		)
 	)
-	(label "pb4"
-		(at 69.85 157.48 180)
+	(label "left"
+		(at 69.85 132.08 180)
 		(effects
 			(font
@@
 		)
 	)
-	(label "left"
+	(label "right"
 		(at 69.85 134.62 180)
-		(effects
-			(font
-				(size 1.27 1.27)
-			)
-			(justify right bottom)
-		)
-	)
-	(label "right"
-		(at 69.85 132.08 180)
 		(effects
 			(font
@@
 		)
 	)
-	(label "pb5"
-		(at 69.85 160.02 180)
-		(effects
-			(font
-				(size 1.27 1.27)
-			)
-			(justify right bottom)
-		)
-	)
 	(label "MISO"
 		(at 69.85 129.54 180)
@@
 	)
 	(label "MOSI"
-		(at 142.24 161.29 180)
-		(effects
-			(font
-				(size 1.27 1.27)
-			)
-			(justify right bottom)
+		(at 116.84 158.75 0)
+		(effects
+			(font
+				(size 1.27 1.27)
+			)
+			(justify left bottom)
 		)
 	)
@@
 	)
 	(label "left"
-		(at 71.12 41.91 180)
+		(at 71.12 39.37 180)
 		(effects
 			(font
@@
 		)
 	)
-	(label "pb4"
-		(at 116.84 158.75 0)
+	(label "pc0"
+		(at 116.84 161.29 0)
 		(effects
 			(font
@@
 			)
 		)
-		(property "Footprint" "Resistor_THT:R_Axial_DIN0207_L6.3mm_D2.5mm_P10.16mm_Horizontal"
+		(property "Footprint" "Resistor_THT:R_Axial_DIN0207_L6.3mm_D2.5mm_P7.62mm_Horizontal"
 			(at 164.592 72.39 90)
 			(hide yes)
@@
 			)
 		)
-		(property "Footprint" "Resistor_THT:R_Axial_DIN0207_L6.3mm_D2.5mm_P10.16mm_Horizontal"
+		(property "Footprint" "Resistor_THT:R_Axial_DIN0207_L6.3mm_D2.5mm_P7.62mm_Horizontal"
 			(at 120.142 71.12 90)
 			(hide yes)
